File: doc/schematics/workstation/workstation.kicad_sch (KiCad schematic)
At the start: 7 parts

Commit message: Fix schematics.
Connections:
- net at GUR2.3. (VCC): now also GUR2.1. (VCC), GUR2.2. (VCC), GUR2.4. (VCC), XA1.GND1 (GND)
- net at GUR2.1. (VCC): now also XA1.D5
- net at FSR_S1., R1.2: now also XA1.A0
- new net: FSR_S1., GUR2.1. (VCC), GUR2.2. (VCC), GUR2.3. (VCC), GUR2.4. (VCC), R1.1, XA1.5V1 (5V)
- now unconnected: GUR2.2. (VCC), GUR2.2. (VCC), GUR2.4. (VCC), GUR2.4. (VCC)
Other:
- company: (none) -> IADE
- title: (none) -> User Experience of Occupancy Detection System
- moved on the sheet: R1
Changed lines of the file:
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@@
 (kicad_sch (version 20230121) (generator eeschema)
   (paper "A4")
+  (title_block
+    (title "User Experience of Occupancy Detection System")
+    (date "2023-06-05")
+    (rev "1")
+    (company "IADE")
+    (comment 1 "Workstation setup")
+    (comment 2 "Prototype")
+  )
   (junction (at 128.27 115.57) (diameter 0) (color 0 0 0 0)
   )
   (junction (at 130.81 115.57) (diameter 0) (color 0 0 0 0)
   )
+  (junction (at 44.45 115.57) (diameter 0) (color 0 0 0 0)
+  )
   (junction (at 124.46 115.57) (diameter 0) (color 0 0 0 0)
   )
-  (junction (at 68.58 100.33) (diameter 0) (color 0 0 0 0)
+  (junction (at 172.72 88.9) (diameter 0) (color 0 0 0 0)
+  )
+  (junction (at 172.72 69.85) (diameter 0) (color 0 0 0 0)
   )
   (junction (at 69.85 135.89) (diameter 0) (color 0 0 0 0)
   )
-  (junction (at 172.72 88.9) (diameter 0) (color 0 0 0 0)
-  )
-  (junction (at 172.72 69.85) (diameter 0) (color 0 0 0 0)
-  )
   (junction (at 140.97 45.72) (diameter 0) (color 0 0 0 0)
   )
-  (junction (at 68.58 115.57) (diameter 0) (color 0 0 0 0)
+  (junction (at 44.45 100.33) (diameter 0) (color 0 0 0 0)
   )
   (wire (pts (xy 124.46 69.85) (xy 134.62 69.85))
@@
     (stroke (width 0) (type default))
   )
-  (wire (pts (xy 68.58 135.89) (xy 68.58 115.57))
+  (wire (pts (xy 44.45 135.89) (xy 44.45 115.57))
     (stroke (width 0) (type default))
   )
@@
     (stroke (width 0) (type default))
   )
-  (wire (pts (xy 68.58 115.57) (xy 124.46 115.57))
-    (stroke (width 0) (type default))
-  )
   (wire (pts (xy 172.72 88.9) (xy 172.72 107.95))
     (stroke (width 0) (type default))
@@
     (stroke (width 0) (type default))
   )
-  (wire (pts (xy 68.58 100.33) (xy 68.58 46.99))
+  (wire (pts (xy 44.45 100.33) (xy 44.45 41.91))
     (stroke (width 0) (type default))
   )
@@
     (stroke (width 0) (type default))
   )
-  (wire (pts (xy 68.58 100.33) (xy 73.66 100.33))
-    (stroke (width 0) (type default))
-  )
   (wire (pts (xy 66.04 45.72) (xy 140.97 45.72))
     (stroke (width 0) (type default))
   )
+  (wire (pts (xy 44.45 100.33) (xy 73.66 100.33))
+    (stroke (width 0) (type default))
+  )
   (wire (pts (xy 124.46 115.57) (xy 128.27 115.57))
     (stroke (width 0) (type default))
@@
     (stroke (width 0) (type default))
   )
+  (wire (pts (xy 69.85 135.89) (xy 140.97 135.89))
+    (stroke (width 0) (type default))
+  )
   (wire (pts (xy 140.97 93.98) (xy 140.97 88.9))
     (stroke (width 0) (type default))
   )
-  (wire (pts (xy 116.84 135.89) (xy 140.97 135.89))
-    (stroke (width 0) (type default))
-  )
-  (wire (pts (xy 69.85 135.89) (xy 68.58 135.89))
+  (wire (pts (xy 69.85 87.63) (xy 69.85 135.89))
+    (stroke (width 0) (type default))
+  )
+  (wire (pts (xy 60.96 135.89) (xy 69.85 135.89))
+    (stroke (width 0) (type default))
+  )
+  (wire (pts (xy 44.45 135.89) (xy 53.34 135.89))
     (stroke (width 0) (type default))
   )
@@
     (stroke (width 0) (type default))
   )
-  (wire (pts (xy 109.22 135.89) (xy 69.85 135.89))
-    (stroke (width 0) (type default))
-  )
   (wire (pts (xy 134.62 120.65) (xy 140.97 120.65))
     (stroke (width 0) (type default))
@@
     (stroke (width 0) (type default))
   )
-  (wire (pts (xy 137.16 46.99) (xy 137.16 59.69))
-    (stroke (width 0) (type default))
-  )
-  (wire (pts (xy 69.85 87.63) (xy 69.85 135.89))
+  (wire (pts (xy 137.16 41.91) (xy 137.16 59.69))
     (stroke (width 0) (type default))
   )
@@
     (stroke (width 0) (type default))
   )
-  (wire (pts (xy 68.58 100.33) (xy 68.58 115.57))
-    (stroke (width 0) (type default))
-  )
-  (wire (pts (xy 68.58 46.99) (xy 137.16 46.99))
+  (wire (pts (xy 44.45 115.57) (xy 124.46 115.57))
+    (stroke (width 0) (type default))
+  )
+  (wire (pts (xy 44.45 100.33) (xy 44.45 115.57))
+    (stroke (width 0) (type default))
+  )
+  (wire (pts (xy 44.45 41.91) (xy 137.16 41.91))
     (stroke (width 0) (type default))
   )
@@
     )
   )
-  (symbol (lib_id "Device:R_US") (at 113.03 135.89 90) (unit 1)
+  (symbol (lib_id "Device:R_US") (at 57.15 135.89 90) (unit 1)
     (in_bom yes) (on_board yes) (dnp no) (fields_autoplaced)
-    (property "Reference" "R1" (at 113.03 130.81 90)
-      (effects (font (size 1.27 1.27)))
-    )
-    (property "Value" "10K" (at 113.03 133.35 90)
-      (effects (font (size 1.27 1.27)))
-    )
-    (property "Footprint" "" (at 113.284 134.874 90)
-      (effects (font (size 1.27 1.27)) hide)
-    )
-    (property "Datasheet" "~" (at 113.03 135.89 0)
-      (effects (font (size 1.27 1.27)) hide)
-    )
+    (property "Reference" "R1" (at 57.15 130.81 90)
+      (effects (font (size 1.27 1.27)))
+    )
+    (property "Value" "10K" (at 57.15 133.35 90)
+      (effects (font (size 1.27 1.27)))
+    )
+    (property "Footprint" "" (at 57.404 134.874 90)
+      (effects (font (size 1.27 1.27)) hide)
+    )
+    (property "Datasheet" "~" (at 57.15 135.89 0)
+      (effects (font (size 1.27 1.27)) hide)
+    )
